Commit message: 1.1.0 Release

File: epson_robot_description/models/C12-C1401S/urdf/epson_robot.urdf.xacro (robot description, xacro)
@@ -263,6 +263,6 @@
     <visual>
       <origin
-        xyz="0 -0.824 -1.152"
-        rpy="1.570796 0 0" />
+        xyz="-1.152 0 -0.830"
+        rpy="3.141593 0 1.570796" />
       <geometry>
         <mesh
@@ -272,11 +272,11 @@
         name="">
         <color
-          rgba="1 1 1 1" />
-      </material>
-    </visual>
-    <collision>
-      <origin
-        xyz="0 -0.824 -1.152"
-        rpy="1.570796 0 0" />
+          rgba="0.75 0.75 0.75 1" />
+      </material>
+    </visual>
+    <collision>
+      <origin
+        xyz="-1.152 0 -0.830"
+        rpy="3.141593 0 1.570796" />
       <geometry>
         <mesh
@@ -289,5 +289,5 @@
     <origin
       xyz="0 0.080 0"
-      rpy="0 0 0" />
+      rpy="-1.570796 -1.570796 0" />
     <parent
       link="${LINK_5}" />
@@ -295,5 +295,5 @@
       link="${LINK_6}" />
     <axis
-      xyz="0 -1 0" />
+      xyz="0 0 -1" />
     <limit
       lower="${joint6_limit_min_rad}"

File: epson_robot_description/models/C8-C1401S/urdf/epson_robot.urdf.xacro (robot description, xacro)
@@ -263,6 +263,6 @@
     <visual>
       <origin
-        xyz="0 -0.824 -1.152"
-        rpy="1.570796 0 0" />
+        xyz="-1.152 0 -0.830"
+        rpy="3.141593 0 1.570796" />
       <geometry>
         <mesh
@@ -272,11 +272,11 @@
         name="">
         <color
-          rgba="1 1 1 1" />
-      </material>
-    </visual>
-    <collision>
-      <origin
-        xyz="0 -0.824 -1.152"
-        rpy="1.570796 0 0" />
+          rgba="0.75 0.75 0.75 1" />
+      </material>
+    </visual>
+    <collision>
+      <origin
+        xyz="-1.152 0 -0.830"
+        rpy="3.141593 0 1.570796" />
       <geometry>
         <mesh
@@ -289,5 +289,5 @@
     <origin
       xyz="0 0.080 0"
-      rpy="0 0 0" />
+      rpy="-1.570796 -1.570796 0" />
     <parent
       link="${LINK_5}" />
@@ -295,5 +295,5 @@
       link="${LINK_6}" />
     <axis
-      xyz="0 -1 0" />
+      xyz="0 0 -1" />
     <limit
       lower="${joint6_limit_min_rad}"

File: epson_robot_description/models/C8-C901S/urdf/epson_robot.urdf.xacro (robot description, xacro)
@@ -263,6 +263,6 @@
     <visual>
       <origin
-        xyz="0 -0.580 -0.902"
-        rpy="1.570796 0 0" />
+        xyz="-0.902 0 -0.580"
+        rpy="3.141593 0 1.570796" />
       <geometry>
         <mesh
@@ -272,11 +272,11 @@
         name="">
         <color
-          rgba="1 1 1 1" />
-      </material>
-    </visual>
-    <collision>
-      <origin
-        xyz="0 -0.580 -0.902"
-        rpy="1.570796 0 0" />
+          rgba="0.75 0.75 0.75 1" />
+      </material>
+    </visual>
+    <collision>
+      <origin
+        xyz="-0.902 0 -0.580"
+        rpy="3.141593 0 1.570796" />
       <geometry>
         <mesh
@@ -289,5 +289,5 @@
     <origin
       xyz="0 0.080 0"
-      rpy="0 0 0" />
+      rpy="-1.570796 -1.570796 0" />
     <parent
       link="${LINK_5}" />
@@ -295,5 +295,5 @@
       link="${LINK_6}" />
     <axis
-      xyz="0 -1 0" />
+      xyz="0 0 -1" />
     <limit
       lower="${joint6_limit_min_rad}"

File: epson_robot_description/models/GX4-C251S/urdf/epson_robot.urdf.xacro (robot description, xacro)
@@ -143,5 +143,5 @@
         name="">
         <color
-          rgba="1 1 1 1" />
+          rgba="0.75 0.75 0.75 1" />
       </material>
     </visual>
@@ -186,5 +186,5 @@
         name="">
         <color
-          rgba="1 1 1 1" />
+          rgba="0.75 0.75 0.75 1" />
       </material>
     </visual>

File: epson_robot_description/models/GX4-C301S/urdf/epson_robot.urdf.xacro (robot description, xacro)
@@ -143,5 +143,5 @@
         name="">
         <color
-          rgba="1 1 1 1" />
+          rgba="0.75 0.75 0.75 1" />
       </material>
     </visual>
@@ -186,5 +186,5 @@
         name="">
         <color
-          rgba="1 1 1 1" />
+          rgba="0.75 0.75 0.75 1" />
       </material>
     </visual>

File: epson_robot_description/models/GX4-C351S-L/urdf/epson_robot.urdf.xacro (robot description, xacro)
@@ -143,5 +143,5 @@
         name="">
         <color
-          rgba="1 1 1 1" />
+          rgba="0.75 0.75 0.75 1" />
       </material>
     </visual>
@@ -186,5 +186,5 @@
         name="">
         <color
-          rgba="1 1 1 1" />
+          rgba="0.75 0.75 0.75 1" />
       </material>
     </visual>

File: epson_robot_description/models/GX4-C351S-R/urdf/epson_robot.urdf.xacro (robot description, xacro)
@@ -143,5 +143,5 @@
         name="">
         <color
-          rgba="1 1 1 1" />
+          rgba="0.75 0.75 0.75 1" />
       </material>
     </visual>
@@ -186,5 +186,5 @@
         name="">
         <color
-          rgba="1 1 1 1" />
+          rgba="0.75 0.75 0.75 1" />
       </material>
     </visual>

File: epson_robot_description/models/GX4-C351S/urdf/epson_robot.urdf.xacro (robot description, xacro)
@@ -143,5 +143,5 @@
         name="">
         <color
-          rgba="1 1 1 1" />
+          rgba="0.75 0.75 0.75 1" />
       </material>
     </visual>
@@ -186,5 +186,5 @@
         name="">
         <color
-          rgba="1 1 1 1" />
+          rgba="0.75 0.75 0.75 1" />
       </material>
     </visual>

File: epson_robot_moveit_config/models/GX4-C251S/srdf/epson_robot.srdf.xacro (robot description, xacro)
@@ -14,9 +14,9 @@
     </group>
     <disable_collisions link1="base_link" link2="j1_link" reason="Adjacent" />
-    <disable_collisions link1="base_link" link2="j2_link" reason="Never" />
-    <disable_collisions link1="base_link" link2="j3_link" reason="Never" />
     <disable_collisions link1="j1_link" link2="j2_link" reason="Adjacent" />
     <disable_collisions link1="j1_link" link2="j3_link" reason="Never" />
+    <disable_collisions link1="j1_link" link2="j4_link" reason="Never" />
     <disable_collisions link1="j2_link" link2="j3_link" reason="Adjacent" />
+    <disable_collisions link1="j2_link" link2="j3_link" reason="Never" />
     <disable_collisions link1="j2_link" link2="j4_link" reason="Never" />
     <disable_collisions link1="j3_link" link2="j4_link" reason="Adjacent" />

File: epson_robot_moveit_config/models/GX4-C301S/srdf/epson_robot.srdf.xacro (robot description, xacro)
@@ -14,9 +14,9 @@
     </group>
     <disable_collisions link1="base_link" link2="j1_link" reason="Adjacent" />
-    <disable_collisions link1="base_link" link2="j2_link" reason="Never" />
-    <disable_collisions link1="base_link" link2="j3_link" reason="Never" />
     <disable_collisions link1="j1_link" link2="j2_link" reason="Adjacent" />
     <disable_collisions link1="j1_link" link2="j3_link" reason="Never" />
+    <disable_collisions link1="j1_link" link2="j4_link" reason="Never" />
     <disable_collisions link1="j2_link" link2="j3_link" reason="Adjacent" />
+    <disable_collisions link1="j2_link" link2="j3_link" reason="Never" />
     <disable_collisions link1="j2_link" link2="j4_link" reason="Never" />
     <disable_collisions link1="j3_link" link2="j4_link" reason="Adjacent" />

File: epson_robot_moveit_config/models/GX4-C351S-L/srdf/epson_robot.srdf.xacro (robot description, xacro)
@@ -14,9 +14,10 @@
     </group>
     <disable_collisions link1="base_link" link2="j1_link" reason="Adjacent" />
-    <disable_collisions link1="base_link" link2="j2_link" reason="Never" />
-    <disable_collisions link1="base_link" link2="j3_link" reason="Never" />
+    <disable_collisions link1="base_link" link2="j1_link" reason="Adjacent" />
     <disable_collisions link1="j1_link" link2="j2_link" reason="Adjacent" />
     <disable_collisions link1="j1_link" link2="j3_link" reason="Never" />
+    <disable_collisions link1="j1_link" link2="j4_link" reason="Never" />
     <disable_collisions link1="j2_link" link2="j3_link" reason="Adjacent" />
+    <disable_collisions link1="j2_link" link2="j3_link" reason="Never" />
     <disable_collisions link1="j2_link" link2="j4_link" reason="Never" />
     <disable_collisions link1="j3_link" link2="j4_link" reason="Adjacent" />

File: epson_robot_moveit_config/models/GX4-C351S-R/srdf/epson_robot.srdf.xacro (robot description, xacro)
@@ -14,9 +14,9 @@
     </group>
     <disable_collisions link1="base_link" link2="j1_link" reason="Adjacent" />
-    <disable_collisions link1="base_link" link2="j2_link" reason="Never" />
-    <disable_collisions link1="base_link" link2="j3_link" reason="Never" />
     <disable_collisions link1="j1_link" link2="j2_link" reason="Adjacent" />
     <disable_collisions link1="j1_link" link2="j3_link" reason="Never" />
+    <disable_collisions link1="j1_link" link2="j4_link" reason="Never" />
     <disable_collisions link1="j2_link" link2="j3_link" reason="Adjacent" />
+    <disable_collisions link1="j2_link" link2="j3_link" reason="Never" />
     <disable_collisions link1="j2_link" link2="j4_link" reason="Never" />
     <disable_collisions link1="j3_link" link2="j4_link" reason="Adjacent" />

File: epson_robot_moveit_config/models/GX4-C351S/srdf/epson_robot.srdf.xacro (robot description, xacro)
@@ -14,9 +14,9 @@
     </group>
     <disable_collisions link1="base_link" link2="j1_link" reason="Adjacent" />
-    <disable_collisions link1="base_link" link2="j2_link" reason="Never" />
-    <disable_collisions link1="base_link" link2="j3_link" reason="Never" />
     <disable_collisions link1="j1_link" link2="j2_link" reason="Adjacent" />
     <disable_collisions link1="j1_link" link2="j3_link" reason="Never" />
+    <disable_collisions link1="j1_link" link2="j4_link" reason="Never" />
     <disable_collisions link1="j2_link" link2="j3_link" reason="Adjacent" />
+    <disable_collisions link1="j2_link" link2="j3_link" reason="Never" />
     <disable_collisions link1="j2_link" link2="j4_link" reason="Never" />
     <disable_collisions link1="j3_link" link2="j4_link" reason="Adjacent" />
